File: Hardware/PCB/EAGLE/Jacdaptor_FeatherWing.brd (EAGLE design)
At the start: 50.8 x 22.9 mm, 27 parts, among them J1 SWD-ADAPTER-, U1 BAT54S,235, U2 STM32G030F6P6, U3 APL3511D

Commit message: Updated design
Parts:
- C1, C2: value 4.7pF -> 4.7uF
Changed lines of the file:
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@@
 <drawing>
 <settings>
-<setting alwaysvectorfont="yes"/>
+<setting alwaysvectorfont="no"/>
 <setting keepoldvectorfont="yes"/>
 <setting verticaltext="up"/>
@@
 <attribute name="NAME" x="32.2" y="9.3" size="0.6096" layer="25" ratio="15" rot="R90" align="bottom-center"/>
 </element>
-<element name="C1" library="milador_SMD" library_urn="urn:adsk.eagle:library:27847482" package="0603" package3d_urn="urn:adsk.eagle:package:29222124/2" value="4.7pF" x="26.3" y="4.3" smashed="yes">
+<element name="C1" library="milador_SMD" library_urn="urn:adsk.eagle:library:27847482" package="0603" package3d_urn="urn:adsk.eagle:package:29222124/2" value="4.7uF" x="26.3" y="4.3" smashed="yes">
 <attribute name="NAME" x="26.3" y="5.062" size="0.6096" layer="25" font="vector" ratio="20" align="bottom-center"/>
 <attribute name="VALUE" x="26.3" y="3.538" size="0.6096" layer="27" font="vector" ratio="20" align="top-center"/>
 </element>
-<element name="C2" library="milador_SMD" library_urn="urn:adsk.eagle:library:27847482" package="0603" package3d_urn="urn:adsk.eagle:package:29222124/2" value="4.7pF" x="35.5" y="18.45" smashed="yes">
+<element name="C2" library="milador_SMD" library_urn="urn:adsk.eagle:library:27847482" package="0603" package3d_urn="urn:adsk.eagle:package:29222124/2" value="4.7uF" x="35.5" y="18.45" smashed="yes">
 <attribute name="NAME" x="35.5" y="19.212" size="0.6096" layer="25" font="vector" ratio="20" align="bottom-center"/>
 <attribute name="VALUE" x="35.5" y="17.688" size="0.6096" layer="27" font="vector" ratio="20" align="top-center"/>
