File: Hardware/PCB/EAGLE/Jacdaptor_FeatherWing-RevB.brd (EAGLE design)
At the start: 50.8 x 22.9 mm, 27 parts, among them J1 SWD-ADAPTER-, U1 BAT54S,235, U2 STM32G030F6P6, U3 APL3511D

Commit message: Updated design RevB
Parts:
- removed H1, H2, H3, H4: MOUNTINGHOLE2.5, milador:MOUNTINGHOLE_2.5_PLATED
- removed U3: APL3511D, milador_SMD:SOT23-5
- added IC1: STM32G030F8P6, milador_SMD:SOP65P640X120-20N
- added J2: (no value), milador:M3-HOLE-PWR
- added J3, J4: (no value), milador:M3-HOLE-GND
- added J5: SWD-ADAPTER-, milador:SWD-ADAPTER
- D1, D2: value DIODE-ZENER-AA-RCLAMP0521PATCT -> RCLAMP0521PATCT
- D3: value (none) -> FM-B2020RGBA
- J1: value SWD-ADAPTER- -> (none); device milador:SWD-ADAPTER -> milador:M3-HOLE-DATA
- U1: value BAT54S,235 -> BAT54S,235-23-3
- U2: value STM32G030F6P6 -> APL3511D; device milador_SMD:TSSOP20 -> milador_SMD:SOT23-5
- moved J1 24.1 mm to (2.54, 20.3), turned to 0 degrees
- moved U2 7.61 mm to (30.4, 16.5)
- turned U1 to 90 degrees
Connections:
- net +3V3: now also IC1.4, J5.1; no longer J1.1, U2.4
- net CS: now also IC1.10; no longer U2.10
- net FAULT: now also IC1.11, U2.1; no longer U2.11, U3.1
- net GND: now also IC1.5, J3.H, J4.H, J5.3, U2.2; no longer H3.P$1, H4.P$1, J1.3, U2.5, U3.2
- net JD: now also IC1.20; no longer U2.20
- net JD5V: now also J2.H; no longer H1.P$1
- net JDF: now also J1.H; no longer H2.P$1
- net LED_B: now also IC1.1; no longer U2.1
- net LED_G: now also IC1.14; no longer U2.14
- net LED_R: now also IC1.15; no longer U2.15
- net LIM: now also IC1.3; no longer U3.3
- net MISO: now also IC1.13; no longer U2.13
- net MOSI: now also IC1.9; no longer U2.9
- net OUT: now also U2.5; no longer U3.5
- net RESET: now also IC1.6, J5.5; no longer J1.5, U2.6
- net RX_RD: now also IC1.12; no longer U2.12
- net SCK: now also IC1.8; no longer U2.8
- net SCL: now also IC1.16; no longer U2.16
- net SDA: now also IC1.17; no longer U2.17
- net SWCLK: now also IC1.19, J5.4; no longer J1.4, U2.19
- net SWDIO: now also IC1.18, J5.2; no longer J1.2, U2.18
- net TX_RD: now also IC1.7; no longer U2.7
- net VUSB: now also U2.4; no longer U3.4
Routing:
- net LED_B: track 8.74 -> 10.1 mm
- net GND: track 149.1 -> 150.3 mm
Other:
- outline, holes or cut-outs redrawn
- board text removed: "5V"
- board text removed: "GND"
- board text removed: "JD"
